File: Kicad/m4live_ctrl_frontpanel.kicad_pcb (KiCad board)
At the start: 4 copper layers, 25 x 128.5 mm, 0 parts

Commit message: Final pcb and frontpanel
Other:
- outline, holes or cut-outs redrawn
- board text added: "M4"
- board text added: "live"
- board text added: "lytrix"
- board text removed: "I"
- board text removed: "X"
- board text removed: "Y"
- board text removed: "m4live"
